File: analog_synth.kicad_pcb (KiCad board)
At the start: 2 copper layers, 0 parts

Commit message: eliminato:              adsr.kicad_pcb     eliminato:              adsr.kicad_pro 	modificato:             analog_synth.kicad_pcb 	nuovo file:             analog_synth.net 	eliminato:              audio_mixer.kicad_pcb 	eliminato:              audio_mixer.kicad_pro 	eliminato:              key_encoder.kicad_pcb 	eliminato:              key_encoder.kicad_pro 	modificato:             key_encoder.kicad_sch 	eliminato:              lfo.kicad_pcb 	eliminato:              lfo.kicad_pro 	eliminato:              noise_gen.kicad_pcb 	eliminato:              noise_gen.kicad_pro 	eliminato:              vca.kicad_pcb 	eliminato:              vca.kicad_prl 	eliminato:              vca.kicad_pro 	modificato:             vca.kicad_sch 	eliminato:              vca.net 	eliminato:              vcf.kicad_pcb 	eliminato:              vcf.kicad_prl 	eliminato:              vcf.kicad_pro 	modificato:             vcf.kicad_sch 	eliminato:              vco.kicad_pcb 	eliminato:              vco.kicad_pro
Parts:
- added D1: 1N4148, Diode_THT:D_DO-35_SOD27_P7.62mm_Horizontal, F.Cu at (194.2, 130.2)
- added D2: 1N4148, Diode_THT:D_DO-35_SOD27_P7.62mm_Horizontal, F.Cu at (126.2, 181.6)
- added R1: 100k, Resistor_SMD:R_0805_2012Metric, F.Cu at (194.9, 112.2)
- added R10: 470k, Resistor_SMD:R_0805_2012Metric, F.Cu at (199.3, 121.1)
- added R11: 8.2k, Resistor_SMD:R_0805_2012Metric, F.Cu at (199.3, 124.0)
- added R12: 22k, Resistor_SMD:R_0805_2012Metric, F.Cu at (199.3, 127.0)
- added R13: 12k, Resistor_SMD:R_0805_2012Metric, F.Cu at (203.7, 112.2)
- added R14: 12k, Resistor_SMD:R_0805_2012Metric, F.Cu at (203.7, 115.2)
- added R15: 4.7k, Resistor_SMD:R_0805_2012Metric, F.Cu at (203.7, 118.2)
- added R16: 12k, Resistor_SMD:R_0805_2012Metric, F.Cu at (203.7, 121.1)
- added R17: 12k, Resistor_SMD:R_0805_2012Metric, F.Cu at (203.7, 124.0)
- added R18: 12k, Resistor_SMD:R_0805_2012Metric, F.Cu at (203.7, 127.0)
- added R19: 3.3m, Resistor_SMD:R_0805_2012Metric, F.Cu at (208.1, 112.2)
- added R2: 22k, Resistor_SMD:R_0805_2012Metric, F.Cu at (194.9, 115.2)
- added R20: 47k, Resistor_SMD:R_0805_2012Metric, F.Cu at (208.1, 115.2)
- added R21: 12k, Resistor_SMD:R_0805_2012Metric, F.Cu at (208.1, 118.2)
- added R22: 470k, Resistor_SMD:R_0805_2012Metric, F.Cu at (208.1, 121.1)
- added R23: 10k, Resistor_SMD:R_0805_2012Metric, F.Cu at (208.1, 124.0)
- added R24: 22k, Resistor_SMD:R_0805_2012Metric, F.Cu at (208.1, 127.0)
- added R25: 330, Resistor_SMD:R_0805_2012Metric, F.Cu at (190.1, 113.0)
- added R26: 470k, Resistor_SMD:R_0805_2012Metric, F.Cu at (212.5, 115.2)
- added R27: 330, Resistor_SMD:R_0805_2012Metric, F.Cu at (212.5, 118.2)
- added R28: 3.3k, Resistor_SMD:R_0805_2012Metric, F.Cu at (212.5, 121.1)
- added R29: 270k, Resistor_SMD:R_0805_2012Metric, F.Cu at (198.2, 205.8)
- added R3: 22k, Resistor_SMD:R_0805_2012Metric, F.Cu at (194.9, 118.2)
- added R30: 270k, Resistor_SMD:R_0805_2012Metric, F.Cu at (201.2, 205.8)
- added R31: 270k, Resistor_SMD:R_0805_2012Metric, F.Cu at (204.1, 205.8)
- added R32: 150k, Resistor_SMD:R_0805_2012Metric, F.Cu at (207.1, 205.8)
- added R33: 470k, Resistor_SMD:R_0805_2012Metric, F.Cu at (210.0, 205.8)
- added R34: 470k, Resistor_SMD:R_0805_2012Metric, F.Cu at (198.2, 201.4)
- added R35: 330, Resistor_SMD:R_0805_2012Metric, F.Cu at (201.2, 201.4)
- added R36: 330, Resistor_SMD:R_0805_2012Metric, F.Cu at (204.1, 201.4)
- added R37: 150k, Resistor_SMD:R_0805_2012Metric, F.Cu at (207.1, 201.4)
- added R38: 10k, Resistor_SMD:R_0805_2012Metric, F.Cu at (69.2, 180.0)
- added R39: 10k, Resistor_SMD:R_0805_2012Metric, F.Cu at (72.2, 180.0)
- added R4: 100k, Resistor_SMD:R_0805_2012Metric, F.Cu at (194.9, 121.1)
- added R40: 470k, Resistor_SMD:R_0805_2012Metric, F.Cu at (75.2, 180.0)
- added R41: 10k, Resistor_SMD:R_0805_2012Metric, F.Cu at (78.1, 180.0)
- added R42: 100k, Resistor_SMD:R_0805_2012Metric, F.Cu at (117.0, 181.0)
- added R43: 10k, Resistor_SMD:R_0805_2012Metric, F.Cu at (84.0, 180.0)
- added R44: 470, Resistor_SMD:R_0805_2012Metric, F.Cu at (122.9, 181.0)
- added R45: 10k, Resistor_SMD:R_0805_2012Metric, F.Cu at (105.2, 176.6)
- added R46: 100k, Resistor_SMD:R_0805_2012Metric, F.Cu at (108.2, 176.6)
- added R47: 1m, Resistor_SMD:R_0805_2012Metric, F.Cu at (111.1, 176.6)
- added R48: 47k, Resistor_SMD:R_0805_2012Metric, F.Cu at (114.0, 176.6)
- added R49: 47k, Resistor_SMD:R_0805_2012Metric, F.Cu at (117.0, 176.6)
- added R5: 100k, Resistor_SMD:R_0805_2012Metric, F.Cu at (194.9, 124.0)
- added R50: 10k, Potentiometer_THT:Potentiometer_Bourns_3009P_Horizontal, F.Cu at (82.2, 140.1)
- added R51: 47k, Resistor_SMD:R_0805_2012Metric, F.Cu at (120.0, 176.6)
- added R52: 20k, Potentiometer_THT:Potentiometer_Bourns_3009P_Horizontal, F.Cu at (82.2, 146.5)
- added R53: 100k, Resistor_SMD:R_0805_2012Metric, F.Cu at (122.9, 176.6)
- added R54: 47k, Resistor_SMD:R_0805_2012Metric, F.Cu at (105.2, 172.2)
- added R55: 10k, Potentiometer_THT:Potentiometer_Bourns_3009P_Horizontal, F.Cu at (82.2, 152.9)
- added R56: 10k, Resistor_SMD:R_0805_2012Metric, F.Cu at (108.2, 172.2)
- added R57: 47k, Resistor_SMD:R_0805_2012Metric, F.Cu at (111.1, 172.2)
- added R58: 20k, Potentiometer_THT:Potentiometer_Bourns_3009P_Horizontal, F.Cu at (82.2, 159.3)
- added R59: 10k, Resistor_SMD:R_0805_2012Metric, F.Cu at (114.0, 172.2)
- added R6: 100k, Resistor_SMD:R_0805_2012Metric, F.Cu at (194.9, 127.0)
- added R60: 47k, Resistor_SMD:R_0805_2012Metric, F.Cu at (117.0, 172.2)
- added R61: 20k, Potentiometer_THT:Potentiometer_Bourns_3009P_Horizontal, F.Cu at (82.2, 165.7)
- added R62: 5.6k, Resistor_SMD:R_0805_2012Metric, F.Cu at (120.0, 172.2)
- added R63: 47k, Resistor_SMD:R_0805_2012Metric, F.Cu at (122.9, 172.2)
- added R64: 20k, Potentiometer_THT:Potentiometer_Bourns_3009P_Horizontal, F.Cu at (82.2, 172.1)
- added R65: 10k, Resistor_SMD:R_0805_2012Metric, F.Cu at (105.2, 167.8)
- added R66: 47k, Resistor_SMD:R_0805_2012Metric, F.Cu at (108.2, 167.8)
- added R67: 47k, Resistor_SMD:R_0805_2012Metric, F.Cu at (111.1, 167.8)
- added R68: 47k, Resistor_SMD:R_0805_2012Metric, F.Cu at (114.0, 167.8)
- added R69: 47k, Resistor_SMD:R_0805_2012Metric, F.Cu at (117.0, 167.8)
- added R7: 100k, Resistor_SMD:R_0805_2012Metric, F.Cu at (199.3, 112.2)
- added R8: 12k, Resistor_SMD:R_0805_2012Metric, F.Cu at (199.3, 115.2)
- added R9: 47k, Resistor_SMD:R_0805_2012Metric, F.Cu at (199.3, 118.2)
- added RV1: 47k, Resistor_SMD:R_0805_2012Metric, F.Cu at (212.5, 124.0)
- added RV2: 10k, Resistor_SMD:R_0805_2012Metric, F.Cu at (212.5, 127.0)
- added RV3: 100k, Resistor_SMD:R_0805_2012Metric, F.Cu at (210.0, 201.4)
- added RV4: 100k, Resistor_SMD:R_0805_2012Metric, F.Cu at (120.0, 167.8)
- added U1: LM301, Package_DIP:DIP-8_W7.62mm_Socket, F.Cu at (139.4, 99.4)
- added U10: 4049, Package_DIP:DIP-14_W7.62mm_Socket, F.Cu at (66.2, 193.8)
- added U11: 4023, Package_DIP:DIP-14_W7.62mm_Socket, F.Cu at (78.0, 193.8)
- added U12: CD4051B, Package_DIP:DIP-16_W7.62mm_Socket, F.Cu at (66.2, 213.2)
- added U13: 4042, Package_DIP:DIP-14_W7.62mm_Socket, F.Cu at (89.7, 193.8)
- added U14: 4042, Package_DIP:DIP-14_W7.62mm_Socket, F.Cu at (101.4, 193.8)
- added U15: CD4051B, Package_DIP:DIP-16_W7.62mm_Socket, F.Cu at (78.0, 213.2)
- added U16: 4024, Package_DIP:DIP-14_W7.62mm_Socket, F.Cu at (113.1, 193.8)
- added U17: 4001, Package_DIP:DIP-14_W7.62mm_Socket, F.Cu at (124.8, 193.8)
- added U18: 4001, Package_DIP:DIP-14_W7.62mm_Socket, F.Cu at (136.5, 193.8)
- added U19: 4001, Package_DIP:DIP-14_W7.62mm_Socket, F.Cu at (148.2, 193.8)
- added U2: LM301, Package_DIP:DIP-8_W7.62mm_Socket, F.Cu at (152.2, 99.2)
- added U20: LM324, Package_DIP:DIP-14_W7.62mm_Socket, F.Cu at (159.9, 193.8)
- added U3: LM301, Package_DIP:DIP-8_W7.62mm_Socket, F.Cu at (165.2, 99.2)
- added U4: LM1496, Package_DIP:DIP-14_W7.62mm_Socket, F.Cu at (165.1, 113.5)
- added U5: LM301, Package_DIP:DIP-8_W7.62mm_Socket, F.Cu at (178.4, 99.4)
- added U6: LM301, Package_DIP:DIP-8_W7.62mm_Socket, F.Cu at (189.4, 182.4)
- added U7: CA3080A, Package_DIP:DIP-8_W7.62mm_Socket, F.Cu at (200.2, 182.4)
- added U8: CA3080A, Package_DIP:DIP-8_W7.62mm_Socket, F.Cu at (211.0, 182.4)
- added U9: LM324, Package_DIP:DIP-14_W7.62mm_Socket, F.Cu at (229.4, 181.8)
