File: analog_synth.kicad_pcb (KiCad board)
At the start: 2 copper layers, 95 parts, among them U1 LM301, U10 4049, U11 4023, U12 CD4051B, U13 4042, U14 4042, U15 CD4051B, U16 4024, U17 4001, U18 4001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

Commit message: modificato:             analog_synth.kicad_pcb 	modificato:             key_encoder.kicad_sch
Parts:
- added U21: CD4066BE, Package_DIP:DIP-14_W7.62mm_Socket, F.Cu at (95.4, 124.3)
- added U22: CD4066BE, Package_DIP:DIP-14_W7.62mm_Socket, F.Cu at (95.2, 146.8)
Connections:
- R50 pad 2: unconnected-(R50-Pad2) -> Net-(R50-Pad2)
- R52 pad 2: unconnected-(R52-Pad2) -> Net-(R52-Pad2)
- R55 pad 2: unconnected-(R55-Pad2) -> Net-(R55-Pad2)
- R58 pad 2: unconnected-(R58-Pad2) -> Net-(R58-Pad2)
- R61 pad 2: unconnected-(R61-Pad2) -> Net-(R61-Pad2)
- R64 pad 2: unconnected-(R64-Pad2) -> Net-(R64-Pad2)
- U11 pad 11: unconnected-(U11-Pad11) -> Net-(U12-C)
- U11 pad 12: unconnected-(U11-Pad12) -> Net-(U12-B)
- U11 pad 13: unconnected-(U11-Pad13) -> Net-(U15-A)
- U12 pad 10: unconnected-(U12-B-Pad10) -> Net-(U12-B)
- U12 pad 11: unconnected-(U12-A-Pad11) -> Net-(U12-A)
- U12 pad 9: unconnected-(U12-C-Pad9) -> Net-(U12-C)
- U13 pad 13: unconnected-(U13-Pad13) -> Net-(U12-B)
- U13 pad 14: unconnected-(U13-Pad14) -> Net-(U12-C)
- U13 pad 4: unconnected-(U13-Pad4) -> Net-(U15-C)
- U13 pad 5: unconnected-(U13-E0-Pad5) -> Net-(U13-E0)
- U13 pad 6: unconnected-(U13-E1-Pad6) -> GNDREF
- U13 pad 7: unconnected-(U13-Pad7) -> Net-(U12-A)
- U13 pad 8: unconnected-(U13-Vss-Pad8) -> GNDREF
- U14 pad 4: unconnected-(U14-Pad4) -> Net-(U15-A)
- U14 pad 5: unconnected-(U14-E0-Pad5) -> Net-(U13-E0)
- U14 pad 6: unconnected-(U14-E1-Pad6) -> GNDREF
- U14 pad 7: unconnected-(U14-Pad7) -> Net-(U15-B)
- U14 pad 8: unconnected-(U14-Vss-Pad8) -> GNDREF
- U15 pad 10: unconnected-(U15-B-Pad10) -> Net-(U15-B)
- U15 pad 11: unconnected-(U15-A-Pad11) -> Net-(U15-A)
- U15 pad 6: unconnected-(U15-INH-Pad6) -> Net-(U15-INH)
- U15 pad 9: unconnected-(U15-C-Pad9) -> Net-(U15-C)
- U16 pad 1: Net-(U16-~{CLK}) -> Net-(U15-INH)
- U16 pad 11: unconnected-(U16-Q1-Pad11) -> Net-(U15-B)
- U16 pad 12: unconnected-(U16-Q0-Pad12) -> Net-(U15-A)
- U16 pad 4: unconnected-(U16-Q5-Pad4) -> Net-(U12-C)
- U16 pad 5: unconnected-(U16-Q4-Pad5) -> Net-(U12-B)
- U16 pad 6: unconnected-(U16-Q3-Pad6) -> Net-(U12-A)
- U16 pad 9: unconnected-(U16-Q2-Pad9) -> Net-(U15-C)
- U17 pad 11: Net-(U16-~{CLK}) -> Net-(U15-INH)
- U17 pad 3: Net-(U17-Pad3) -> Net-(U13-E0)
- U17 pad 5: Net-(U17-Pad3) -> Net-(U13-E0)
- U17 pad 6: Net-(U17-Pad3) -> Net-(U13-E0)
- U18 pad 3: Net-(U16-~{CLK}) -> Net-(U15-INH)
- U19 pad 2: Net-(U17-Pad3) -> Net-(U13-E0)
